File: STM_RF_PCB/STM_RF_PCB.kicad_sch (KiCad schematic)
At the start: 43 parts, among them J1 U.FL, J2 USB_B_Micro, J3 SWD STLINk, SW1 UP, SW2 LF, SW3 DN, SW4 RT, SW5 A, SW6 B, U1 nRF24L01P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

Commit message: Added I2C interface back and changed to SMA antenna
Parts:
- added J4: Conn_01x04, symbol Connector_Generic:Conn_01x04
- added R6, R7: 2.2k, symbol Device:R
- J1: value U.FL -> SMA
Connections:
- net +3V3: now also J4.2 (Pin_2), R6.1, R7.1
- net Button_A: now also U4.12 (PA6); no longer U4.18 (PA8)
- net Button_B: now also U4.13 (PA7); no longer U4.19 (PA9)
- net Button_DN: now also U4.9 (PA3); no longer U4.11 (PA5)
- net Button_LF: now also U4.10 (PA4); no longer U4.12 (PA6)
- net Button_RT: now also U4.11 (PA5); no longer U4.13 (PA7)
- net Button_UP: now also U4.8 (PA2); no longer U4.10 (PA4)
- net GND: now also J4.1 (Pin_1)
- net at D1.2 (A): now also U4.6 (PA0); no longer U4.8 (PA2)
- net I2C1_SDA: now reaches U4.20 (PA10)
- net I2C1_SDA: now also J4.4 (Pin_4), R7.2
- net at U4.7 (PA1): now also D2.2 (A)
- new net I2C1_SCL: J4.3 (Pin_3), R6.2, U4.19 (PA9)
- no-connect marks 11 -> 9
Other:
- note added: "I2C Screen"
- moved on the sheet: C13, C14, C15, C16, C17, D1, D2, J3, R3, R4, R5, U4
