File: STM_RF_PCB/STM_RF_PCB.kicad_pcb (KiCad board)
At the start: 0 parts

Commit message: Work on PCB
Parts:
- added C1: 33n, Capacitor_SMD:C_0402_1005Metric, F.Cu at (152.3, 84.5)
- added C10: 1p, Capacitor_SMD:C_0402_1005Metric, F.Cu at (155.1, 90.4)
- added C11: 10u, Capacitor_SMD:C_0603_1608Metric, F.Cu at (45.4, 56.4)
- added C12: 10u, Capacitor_SMD:C_0603_1608Metric, F.Cu at (45.4, 58.9)
- added C13: 100n, Capacitor_SMD:C_0402_1005Metric, F.Cu at (158.0, 84.5)
- added C14: 100n, Capacitor_SMD:C_0402_1005Metric, F.Cu at (158.0, 86.5)
- added C15: 100n, Capacitor_SMD:C_0402_1005Metric, F.Cu at (158.0, 88.4)
- added C16: 100n, Capacitor_SMD:C_0402_1005Metric, F.Cu at (158.0, 90.4)
- added C17: 4.7u, Capacitor_SMD:C_0603_1608Metric, F.Cu at (45.4, 61.4)
- added C2: 10n, Resistor_SMD:R_0603_1608Metric, F.Cu at (45.4, 51.3)
- added C3: 1n, Capacitor_SMD:C_0402_1005Metric, F.Cu at (152.3, 86.5)
- added C4: 4.7u, Capacitor_SMD:C_0603_1608Metric, F.Cu at (45.4, 53.8)
- added C5: 12p, Capacitor_SMD:C_0402_1005Metric, F.Cu at (152.3, 88.4)
- added C6: 12p, Capacitor_SMD:C_0402_1005Metric, F.Cu at (152.3, 90.4)
- added C7: 2.2n, Capacitor_SMD:C_0402_1005Metric, F.Cu at (155.1, 84.5)
- added C8: 4.7p, Capacitor_SMD:C_0402_1005Metric, F.Cu at (155.1, 86.5)
- added C9: 1.5p, Capacitor_SMD:C_0402_1005Metric, F.Cu at (155.1, 88.4)
- added D1: BLUE, LED_SMD:LED_0603_1608Metric, F.Cu at (49.4, 65.4)
- added D2: GREEN, LED_SMD:LED_0603_1608Metric, F.Cu at (49.4, 68.0)
- added F1: 120 mA, Fuse:Fuse_1206_3216Metric, F.Cu at (50.2, 58.0)
- added FB1: 100 @ 100 MHz, Inductor_SMD:L_0805_2012Metric, F.Cu at (49.6, 70.6)
- added J1: SMA, Library:SMA-KWE902, F.Cu at (148.5, 49.0)
- added J2: USB_B_Micro, Library:MICRO-02-G2P3-A1T2, F.Cu at (130.0, 48.2)
- added J3: SWD STLINk, Connector_PinHeader_2.54mm:PinHeader_2x05_P2.54mm_Vertical, F.Cu at (144.4, 129.5)
- added J4: Conn_01x04, Connector_PinSocket_2.54mm:PinSocket_1x04_P2.54mm_Vertical, F.Cu at (174.0, 51.5)
- added L1: 2.7n, Inductor_SMD:L_0402_1005Metric, F.Cu at (49.4, 101.2)
- added L2: 8.2n, Inductor_SMD:L_0402_1005Metric, F.Cu at (49.4, 103.2)
- added L3: 3.9n, Inductor_SMD:L_0402_1005Metric, F.Cu at (49.4, 105.2)
- added R1: 22k, Resistor_SMD:R_0402_1005Metric, F.Cu at (49.4, 107.2)
- added R2: 1M, Resistor_SMD:R_0402_1005Metric, F.Cu at (49.4, 109.2)
- added R3: 10k, Resistor_SMD:R_0402_1005Metric, F.Cu at (49.4, 111.2)
- added R4: 2.2k, Resistor_SMD:R_0603_1608Metric, F.Cu at (45.4, 63.9)
- added R5: 2.2k, Resistor_SMD:R_0603_1608Metric, F.Cu at (45.4, 66.4)
- added R6: 2.2k, Resistor_SMD:R_0603_1608Metric, F.Cu at (45.4, 68.9)
- added R7: 2.2k, Resistor_SMD:R_0603_1608Metric, F.Cu at (45.4, 71.4)
- added SW1: UP, Library:TC-1103-C-D, F.Cu at (89.8, 62.0)
- added SW2: LF, Library:TC-1103-C-D, F.Cu at (63.2, 80.5)
- added SW3: DN, Library:TC-1103-C-D, F.Cu at (89.2, 102.0)
- added SW4: RT, Library:TC-1103-C-D, F.Cu at (115.8, 80.0)
- added SW5: A, Library:TC-1103-C-D, F.Cu at (207.2, 87.0)
- added SW6: B, Library:TC-1103-C-D, F.Cu at (237.2, 70.0)
- added U1: nRF24L01P, Package_DFN_QFN:QFN-20-1EP_4x4mm_P0.5mm_EP2.5x2.5mm, F.Cu at (149.0, 66.5)
- added U2: USBLC6-2SC6, Package_TO_SOT_SMD:SOT-23-6, F.Cu at (121.1, 56.5)
- added U3: XC6206P332MR, Package_TO_SOT_SMD:SOT-23-3, F.Cu at (113.0, 53.0)
- added U4: STM32L432KBUx, Package_DFN_QFN:UFQFPN-32-1EP_5x5mm_P0.5mm_EP3.5x3.5mm, F.Cu at (169.1, 84.9)
- added Y1: 16 MHz, Crystal:Crystal_SMD_3225-4Pin_3.2x2.5mm, F.Cu at (50.0, 61.8)
Other:
- copper layers 0 -> 4
