File: STM_RF_PCB/STM_RF_PCB.kicad_pcb (KiCad board)
At the start: 4 copper layers, 160 x 90 mm, 48 parts, among them J1 SMA, J2 USB_B_Micro, J3 SWD STLINk, J4 Conn_01x04, SW1 UP, SW2 LF, SW3 DN, SW4 RT, SW5 A, SW6 B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

Commit message: PCB work complete + fab outputs
Parts:
- added 3v3: TestPoint_Plated_Hole_D2.0mm, TestPoint:TestPoint_Plated_Hole_D2.0mm, F.Cu at (73.2, 137.0)
- added GND: TestPoint_Plated_Hole_D2.0mm, TestPoint:TestPoint_Plated_Hole_D2.0mm, F.Cu at (78.0, 137.0)
- moved R2 5.81 mm to (193.8, 80.5)
- moved C5 1.77 mm to (197.2, 82.8)
- moved C6 1.77 mm to (191.8, 88.2)
- moved Y1 1.77 mm to (193.0, 83.5)
Routing:
- net GND: track 28.3 -> 35.8 mm, vias 8 -> 15
- net NRF_XC1: track 11.1 -> 8.20 mm
- net NRF_XC2: track 13.8 -> 11.1 mm
- net +3V3: track 55.8 -> 58.4 mm, vias 6 -> 9
- net USB_D+: track 39.3 -> 40.2 mm
- net USB_D-: track 39.4 -> 40.3 mm
Other:
- board text added: "Prasana Ganesh Petar Acimovic University of Cincinnati"
- board text added: "RF_CONTROLLER_UHP"
