File: STM_RF_PCB/STM_RF_PCB.kicad_pcb (KiCad board)
At the start: 4 copper layers, 160 x 90 mm, 50 parts, among them J1 SMA, J2 USB_B_Micro, J3 SWD STLINk, J4 Conn_01x04, SW1 UP, SW2 LF, SW3 DN, SW4 RT, SW5 A, SW6 B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

Commit message: added san jose 2024
Other:
- board text added: "San Jose 2024"
Changed lines of the file:
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@@
+		)
+	)
+	(gr_text "San Jose 2024"
+		(at 226 149.25 0)
+		(layer "B.SilkS")
+		(effects
+			(font
+				(size 2 2)
+				(thickness 0.16)
+			)
+			(justify left bottom mirror)
 		)
 	)

Commit message: Fab outputs
Routing:
- net GND: track 35.8 -> 38.2 mm
Changed lines of the file:
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@@
-	)
-	(segment
-		(start 204.75 76.23)
-		(end 204.75 78)
-		(width 0.3424)
-		(layer "F.Cu")
-		(net 1)
 	)
 	(segment
@@
 	)
 	(segment
-		(start 204.75 78.75)
-		(end 203.75 79.75)
+		(start 205.75 78.5)
+		(end 204.5 79.75)
+		(width 0.3424)
+		(layer "F.Cu")
+		(net 1)
+	)
+	(segment
+		(start 204.5 79.75)
+		(end 202.73 79.75)
 		(width 0.3424)
 		(layer "F.Cu")
@@
 	)
 	(segment
+		(start 204.75 76.23)
+		(end 204.75 77.5)
+		(width 0.3424)
+		(layer "F.Cu")
+		(net 1)
+	)
+	(segment
 		(start 150.25 108.25)
 		(end 151 109)
 		(width 0.25)
+		(layer "F.Cu")
+		(net 1)
+	)
+	(segment
+		(start 204.75 77.5)
+		(end 205.75 78.5)
+		(width 0.3424)
 		(layer "F.Cu")
 		(net 1)
@@
 	)
 	(segment
-		(start 202.73 78)
-		(end 204.75 78)
-		(width 0.3424)
+		(start 198.25 73.5)
+		(end 197.75 73.5)
+		(width 0.25)
 		(layer "F.Cu")
 		(net 1)
 	)
 	(segment
-		(start 198.25 73.5)
-		(end 197.75 73.5)
-		(width 0.25)
+		(start 202.73 78)
+		(end 205.25 78)
+		(width 0.3424)
 		(layer "F.Cu")
 		(net 1)
@@
 		(end 145.5 69)
 		(width 0.25)
-		(layer "F.Cu")
-		(net 1)
-	)
-	(segment
-		(start 203.75 79.75)
-		(end 202.73 79.75)
-		(width 0.3424)
-		(layer "F.Cu")
-		(net 1)
-	)
-	(segment
-		(start 204.75 78)
-		(end 204.75 78.75)
-		(width 0.3424)
 		(layer "F.Cu")
 		(net 1)
@@
 	)
 	(segment
+		(start 205.25 78)
+		(end 205.75 78.5)
+		(width 0.3424)
+		(layer "F.Cu")
+		(net 1)
+	)
+	(segment
 		(start 196.25 75)
 		(end 194.6875 75)
@@
 	)
 	(via
-		(at 204.75 78)
+		(at 205.75 78.5)
 		(size 0.8)
 		(drill 0.4)
